File: kicad/sbc09.kicad_pcb (KiCad board)
At the start: 4 copper layers, 100 x 100 mm, 55 parts, among them J1 Conn_01x04_Male, J2 Conn_01x06_Male, J3 Conn_01x06_Male, J4 Conn_01x06_Male, J6 Conn_02x25_Odd_Even, Q1 2N7000, SW1 SW_Push, U10 74LS670, U11 74LS670, U12 AS6C4008-55PCN, U13 SST39SF040-DIP, U15 XR68C681CJ, U4 MC6809E, U5 74HCT125, U6 ATF22V10C, U7 ATF22V10C, U8 74LS670, U9 74LS670, X1 8MHz, X2 3.6864MHz

Commit message: KiCAD: more work...
Parts:
- removed JP15: Jumper_3_Bridged12, Connector_PinHeader_2.54mm:PinHeader_1x03_P2.54mm_Vertical
- added JP8: Jumper_2_Open, Connector_PinHeader_2.54mm:PinHeader_1x02_P2.54mm_Vertical, F.Cu at (151.9, 39.4)
- added R3: 100R, Resistor_THT:R_Axial_DIN0207_L6.3mm_D2.5mm_P10.16mm_Horizontal, F.Cu at (186.9, 114.9)
- added R5: 3K6, Resistor_THT:R_Axial_DIN0207_L6.3mm_D2.5mm_P10.16mm_Horizontal, F.Cu at (136.7, 40.6)
- moved H4 133.2 mm to (100.3, 49.5)
- moved H1 94.8 mm to (191.8, 141.0)
- moved H2 83.2 mm to (99.7, 141.6)
- moved U9 71.4 mm to (128.3, 48.3)
- moved C10 69.0 mm to (153.0, 48.3), turned to -90 degrees
- moved R1 46.9 mm to (180.8, 114.9)
- moved R4 44.0 mm to (181.6, 65.4), turned to -90 degrees
- moved U5 43.8 mm to (170.2, 101.6)
- moved C4 43.7 mm to (166.4, 101.6)
- moved U4 43.6 mm to (154.9, 101.6)
- moved C7 42.7 mm to (181.6, 124.5)
- moved U7 42.6 mm to (170.2, 124.5)
- moved C6 42.5 mm to (166.4, 124.5)
- moved U6 42.4 mm to (154.9, 124.5)
- moved Q1 42.2 mm to (184.3, 118.5)
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- renumbered C4 to C1, C7 to C10, C15 to C11, C17 to C12, C18 to C13, C12 to C2, C13 to C3, C8 to C4, C9 to C5, C10 to C6, C11 to C7, C5 to C8, C6 to C9, R3 to R4, U4 to U1, U6 to U10, U15 to U11, U12 to U2, U13 to U3, U8 to U4, U9 to U5, U10 to U6, U11 to U7, U5 to U8, U7 to U9
Connections:
- net Net-(J6-Pad27) renamed /VBUS
- C13 pad 2: Net-(C18-Pad2) -> Net-(C13-Pad2)
- Q1 pad 2: Net-(C18-Pad2) -> Net-(C13-Pad2)
- R1 pad 1: Net-(C18-Pad2) -> Net-(R1-Pad1)
- RN2 pad 2: QA15 -> /QA17
- RN2 pad 5: /QA17 -> QA15
- RN3 pad 2: QA19 -> QA21
- RN3 pad 5: QA21 -> QA19
- SW1 pad 1: Net-(C18-Pad2) -> Net-(R1-Pad1)
- U10 pad 10: 16KMODE -> A14TO11
- U10 pad 11: QA19 -> /A15
- U10 pad 14: QA13 -> QA20
- U10 pad 15: /nCSIOINT -> QA21
- U10 pad 16: /nCSUART -> nRW
- U10 pad 17: nWRMMU1 -> /nCSINTIO
- U10 pad 18: nWRMMU0 -> nCSROM
- U10 pad 19: nWR -> nCSRAM
- U10 pad 20: nRD -> nCSEXT
- U10 pad 21: /A8X -> nCSEXTIO
- U10 pad 3: BA -> nENMMU
- U10 pad 4: BS -> RnW
- U10 pad 5: RnW -> /A6
- U10 pad 6: /A4 -> /A7
- U10 pad 7: /A5 -> /A8
- U10 pad 8: /A8 -> /A9
- U10 pad 9: /A13 -> /A10
- U2 pad 24: nRD -> nRW
- U2 pad 25: /A11 -> /A11X
- U2 pad 27: /A8X -> /A8
- U2 pad 29: nWR -> RnW
- U2 pad 3: QA14 -> QA15
- U2 pad 31: QA15 -> QA14
- U3 pad 24: nRD -> nRW
- U3 pad 25: /A11 -> /A11X
- U3 pad 27: /A8X -> /A8
- U3 pad 31: nWR -> Net-(U3-Pad31)
- U9 pad 1: nENMMU -> BA
- U9 pad 10: /A14 -> QA19
- U9 pad 11: /A15 -> nENMMU
- U9 pad 14: nENMMU1 -> /nCSINTIO
- U9 pad 15: nENMMU0 -> A14TO11
- U9 pad 16: /SPARE -> /nCSUART
- U9 pad 17: nCSRAM -> nWRMMU0
- U9 pad 18: nCSROM -> nWRMMU1
- U9 pad 19: nCSEXTIO -> QA13
- U9 pad 2: /A6 -> BS
- U9 pad 20: nCSEXT -> QA14
- U9 pad 21: /nCSIOINT -> /A11X
- U9 pad 22: QA21 -> nENMMU0
- U9 pad 23: QA20 -> nENMMU1
- U9 pad 3: /A7 -> RnW
- U9 pad 4: /A8 -> /A4
- U9 pad 5: /A9 -> /A5
- U9 pad 6: /A10 -> /A11
- U9 pad 7: /A11 -> /A12
- U9 pad 8: /A12 -> /A13
- U9 pad 9: /A13 -> /A14
Routing:
- net nRST: track 185.8 -> 30.1 mm, vias 6 -> 1
- net /A0: track 215.6 -> 63.8 mm, vias 5 -> 2
- net /D0: track 76.1 -> 205.1 mm, vias 1 -> 4
- net 16KMODE: track 123.1 -> 0.00 mm, vias 3 -> 0
- net /A1: track 207.8 -> 86.1 mm, vias 5 -> 4
- net RnW: track 119.2 -> 0.00 mm, vias 6 -> 0
- net /A2: track 174.5 -> 56.2 mm, vias 3 -> 2
- net /D6: track 177.9 -> 294.7 mm, vias 4 -> 8
- net /A15: track 55.4 -> 171.7 mm, vias 2 -> 5
- net /A3: track 161.6 -> 49.3 mm, vias 3 -> 2
- net /A8X: track 104.5 -> 0.00 mm, vias 4 -> 0
- net /A11: track 104.0 -> 0.00 mm, vias 3 -> 0
- net /SDCS: track 102.0 -> 0.00 mm, vias 2 -> 0
- net /SDMOSI: track 95.8 -> 0.00 mm, vias 2 -> 0
- net nENMMU: track 95.0 -> 0.00 mm, vias 2 -> 0
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- added copper zone on In2.Cu, net /VBUS
Other:
- board size 100 x 100 mm -> 101.6 x 101.6 mm
- board text removed: "12MHz"
- board text removed: "28"
- board text removed: "3.6864MHz"
- board text removed: "32"
- board text removed: "6809"
- board text removed: "6809E"
- board text removed: "E"
- board text removed: "QA14"
